File: Hardware/pcb.brd (EAGLE design)
At the start: 170.2 x 111.2 mm, 103 parts, among them IC1 BD5229G-TR, IC4 XC6220A331MR-G, J1 FH34SRJ-24S-0.5SH_99_, J2 SAMACSYS_PARTS_USB4110-GF-A, J3 QWIIC_RIGHT_ANGLE, J4 112A-TAAR-R03_ATTEND, Q1 20V/4.2A/52mΩ/1.4W, Q2 20V/4.2A/52mΩ/1.4W, Q3 SI1308EDL-T1-GE3, U1 W25Q512JVEIQ, U2 ESP32-C6-WROOM-1-N8, U3 DS3231SN#, U4 MAX17048G+T10

Commit message: addressed all issues
Parts:
- moved BOOT_BUTTON 0.81 mm to (24.0, 108.9)
- moved C6 0.80 mm to (27.4, 108.8)
- moved R_BOOT 0.70 mm to (20.6, 108.7)
- moved RESET_BUTTON 0.20 mm to (49.0, 109.0)
Routing:
- net SRC: track 50.9 -> 52.0 mm
- net GND: track 157.4 -> 158.2 mm
- net IO/BOOT: track 55.3 -> 56.0 mm
- net FLASH_CS: track 27.6 -> 27.0 mm
Other:
- outline, holes or cut-outs redrawn
